File: HardWare/full_ac_thermostrat_Mainboard.kicad_pcb (KiCad board)
At the start: 2 copper layers, 255 x 45 mm, 128 parts, among them J1 CON.1X3P5.0MM.WJ103, J2 CON.1X3P5.0MM.WJ103, J3 CON.DIP.1X16P.5.0MM, J4 CON.DIP.1X5P.2.0MM, J6 WJ103, K1 RELAY.HF32F-012-HSL, K2 RELAY.HF32F-012-HSL, K3 RELAY.HF32F-012-HSL, K4 RELAY.HF32F-012-HSL, K5 RELAY.HF32F-012-HSL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

Commit message: 修改WiFi模块  安信可
Parts:
- added CY3: 2.2nF.250V, MenRed_Library_CAP:CAP.DIP.Y.102M／250V, F.Cu at (90.4, 60.1)
- added CY4: 2.2nF.250V, MenRed_Library_CAP:CAP.DIP.Y.102M／250V, F.Cu at (100.5, 59.0)
- added LED1: BL-HG635A, MenRed_Library_DIODE:D.BL-HG635A-TRB-LED, F.Cu at (210.2, 66.2)
- added R34: 39K.0603, MenRed_Library_RES:RES.SMT.0603, F.Cu at (210.3, 69.8)
- D1: value D.SMT.MB10S -> D.SMT.KBS10; footprint MenRed_Library_DIODE:D.SMT.MD6S.TR -> MenRed_Library_DIODE:D.SMT.KBP310G
- EC2, EC4: footprint MenRed_Library_CAP:CAP.DIP.2.2uF／400V.6.3X11 -> MenRed_Library_CAP:CAP.DIP.6.8UF.400V.10MM2
- EC6: value 100uF.25V -> 220uF.25V; footprint MenRed_Library_CAP:CAP.SMT.100UF.25V -> MenRed_Library_CAP:CAP.SMT.220UF.16V
- EC8: footprint MenRed_Library_CAP:CAP.DIP.330uF／25V.8X12 -> MenRed_Library_CAP:CAP.SMT.220UF.16V
- L1: value 20mh -> L.DIP.JF1058T-22MH
- R10, R11: value 10R.0805 -> 1R6.0805
- R7: value 10R.0805 -> 3.6K.0805
- R8: value 10R.0805 -> NC
- moved TR1 5.52 mm to (96.9, 71.2)
- moved R28 5.31 mm to (110.4, 59.0)
- moved C14 4.75 mm to (116.0, 59.1)
- moved C5 4.57 mm to (84.1, 63.3)
- moved D3 4.57 mm to (83.7, 67.5)
- moved D4 4.57 mm to (82.3, 80.0)
- moved EC3 4.57 mm to (76.8, 67.2)
- moved R10 4.57 mm to (73.8, 78.3)
- moved R11 4.57 mm to (73.8, 75.9)
- moved R23 4.57 mm to (84.0, 60.6)
- moved R26 4.57 mm to (79.6, 62.3)
- moved R7 4.57 mm to (73.8, 73.6)
- moved R8 4.57 mm to (73.7, 71.2)
- moved U1 4.57 mm to (80.8, 72.3)
- moved R22 4.57 mm to (79.2, 76.9)
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Connections:
- D1 pad 3: GNDA -> Net-(D1-Pad3)
- D1 pad 4: Net-(D1-Pad4) -> GNDA
- EC2 pad 1: Net-(D1-Pad4) -> Net-(D1-Pad3)
- K2 pad 3: /O_ACT8 -> +12V
- K2 pad 4: +12V -> /O_ACT8
- L4 pad 1: Net-(D1-Pad4) -> Net-(D1-Pad3)
Routing:
- net /AC_N: track 297.9 -> 491.1 mm
- net Net-(CY1-Pad1): track 84.1 -> 156.8 mm
- net Net-(D1-Pad3): track 0.00 -> 69.8 mm
- net GNDA: track 169.8 -> 228.3 mm
- net Net-(CY2-Pad2): track 34.9 -> 80.4 mm
- net Net-(C5-Pad1): track 79.3 -> 112.1 mm
- net Net-(D1-Pad4): track 28.3 -> 0.00 mm
- net GND: track 640.6 -> 663.6 mm, vias 104 -> 102
- net +12V: track 328.5 -> 346.5 mm, vias 2 -> 3
- net Net-(C12-Pad2): track 70.6 -> 87.9 mm
- net Net-(D3-Pad2): track 18.5 -> 29.0 mm
- net /Ch8: track 10.9 -> 20.7 mm
- net /Ch7: track 11.1 -> 20.5 mm
- net /Ch6: track 11.2 -> 20.2 mm
- net /Ch5: track 11.3 -> 20.0 mm
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Other:
- outline, holes or cut-outs redrawn
