File: HardWare/full_ac_thermostrat_Mainboard.sch (KiCad schematic (older format))
At the start: 128 parts, among them J1 CON.1X3P5.0MM.WJ103, J2 CON.1X3P5.0MM.WJ103, J3 CON.DIP.1X16P.5.0MM, J4 CON.DIP.1X5P.2.0MM, J6 WJ103, K1 RELAY.HF32F-012-HSL, K2 RELAY.HF32F-012-HSL, K3 RELAY.HF32F-012-HSL, K4 RELAY.HF32F-012-HSL, K5 RELAY.HF32F-012-HSL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

Commit message: 修改WiFi模块  安信可
Parts:
- added CY3, CY4: 2.2nF.250V, MenRed_Library_CAP:CAP.DIP.Y.102M／250V, symbol MenRed_Library_CAP:CAP.DIP.X.0.1uF.275V
- added LED1: BL-HG635A, MenRed_Library_DIODE:D.BL-HG635A-TRB-LED, symbol MenRed_Library_DIODE:D.LED.SMT.BL-HG635A-TRB-0805
- added R34: 39K.0603, MenRed_Library_RES:RES.SMT.0603, symbol MenRed_Library_RES:RES.SMT.10K.0603
- D1: value D.SMT.MB10S -> D.SMT.KBS10; footprint MenRed_Library_DIODE:D.SMT.MD6S.TR -> MenRed_Library_DIODE:D.SMT.KBP310G
- EC2, EC4: footprint MenRed_Library_CAP:CAP.DIP.2.2uF／400V.6.3X11 -> MenRed_Library_CAP:CAP.DIP.6.8UF.400V.10MM2
- EC6: value 100uF.25V -> 220uF.25V; footprint MenRed_Library_CAP:CAP.SMT.100UF.25V -> MenRed_Library_CAP:CAP.SMT.220UF.16V
- EC8: footprint MenRed_Library_CAP:CAP.DIP.330uF／25V.8X12 -> MenRed_Library_CAP:CAP.SMT.220UF.16V
- L1: value L.DIP.JF1058T-3.5MH -> L.DIP.JF1058T-22MH
- R10, R11: value 10R.0805 -> 1R6.0805
- R7: value 10R.0805 -> 3.6K.0805
- R8: value 10R.0805 -> NC
Connections:
- net +12V: now also K2.3; no longer K2.4
- net +3V3: now also LED1.2 (A)
- net GND: now also R34.1
- net GNDA: now also D1.4 (V-); no longer D1.3 (V+)
- net O_ACT8: now also K2.4; no longer K2.3
- net at C12.2, C6.2, EC5.2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: now also CY4.1
- net at C5.1, EC4.1, L4.2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: now also CY3.2
- net at EC2.1, L4.1: now also D1.3 (V+); no longer D1.4 (V-)
- new net: CY3.1, CY4.2
- new net: LED1.1 (K), R34.2
Changed lines of the file:
@@
 P 9590 1185
 F 0 "EC6" V 9690 1210 50  0000 L CNN
-F 1 "100uF.25V" V 9880 1015 50  0000 L CNN
-F 2 "MenRed_Library_CAP:CAP.SMT.100UF.25V" H 9440 1185 60  0001 C CNN
+F 1 "220uF.25V" V 9880 1015 50  0000 L CNN
+F 2 "MenRed_Library_CAP:CAP.SMT.220UF.16V" H 9440 1185 60  0001 C CNN
 F 3 "" H 9440 1185 60  0000 C CNN
 	1    9590 1185
@@
 F 0 "EC8" V 1495 8075 60  0000 L CNN
 F 1 "100uF.35V" V 1495 8300 60  0000 L CNN
-F 2 "MenRed_Library_CAP:CAP.DIP.330uF／25V.8X12" H 1525 7445 60  0001 C CNN
+F 2 "MenRed_Library_CAP:CAP.SMT.220UF.16V" H 1525 7445 60  0001 C CNN
 F 3 "" H 1450 7720 60  0000 C CNN
 	1    1600 7720
@@
 O_ACT8
 Wire Wire Line
-	1775 8575 1550 8575
-Text Label 1550 8575 0    50   ~ 0
+	2450 8575 2225 8575
+Text Label 2225 8575 0    50   ~ 0
 AC_L
-Text Label 2490 8575 2    50   ~ 0
+Text Label 1775 8575 2    50   ~ 0
 Ch8
 Wire Wire Line
-	2225 8575 2490 8575
+	1510 8575 1775 8575
 $Comp
 L MenRed_Library_BJT:BJT_SMT_SS8050_SOT-23 Q1
@@
 F 3 "" H 1975 8775 50  0001 C CNN
 	1    2000 8775
-	1    0    0    -1
+	-1   0    0    -1
 $EndComp
 $Comp
@@
 F 0 "EC4" V 5365 875 60  0000 L CNN
 F 1 "6.8uF.400V" V 5535 985 60  0000 L CNN
-F 2 "MenRed_Library_CAP:CAP.DIP.2.2uF／400V.6.3X11" H 5295 1175 60  0001 C CNN
+F 2 "MenRed_Library_CAP:CAP.DIP.6.8UF.400V.10MM2" H 5295 1175 60  0001 C CNN
 F 3 "" H 5295 1175 60  0000 C CNN
 	1    5370 1175
@@
 F 0 "EC2" V 4795 875 60  0000 L CNN
 F 1 "6.8uF.400V" V 4960 915 60  0000 L CNN
-F 2 "MenRed_Library_CAP:CAP.DIP.2.2uF／400V.6.3X11" H 4720 1175 60  0001 C CNN
+F 2 "MenRed_Library_CAP:CAP.DIP.6.8UF.400V.10MM2" H 4720 1175 60  0001 C CNN
 F 3 "" H 4720 1175 60  0000 C CNN
 	1    4795 1175
@@
 P 2875 1180
 F 0 "L1" H 2875 899 50  0000 C CNN
-F 1 "L.DIP.JF1058T-3.5MH" H 2875 990 50  0000 C CNN
+F 1 "L.DIP.JF1058T-22MH" H 2875 990 50  0000 C CNN
 F 2 "MenRed_Library_L:L.DIP.JF1058T-3.5MH" H 2975 980 60  0001 C CNN
 F 3 "" H 2975 980 60  0000 C CNN
@@
 P 4245 1175
 F 0 "D1" H 4240 1330 50  0000 C CNN
-F 1 "D.SMT.MB10S" H 4255 1025 50  0000 C CNN
-F 2 "MenRed_Library_DIODE:D.SMT.MD6S.TR" H 3880 1640 50  0001 C CNN
+F 1 "D.SMT.KBS10" H 4255 1025 50  0000 C CNN
+F 2 "MenRed_Library_DIODE:D.SMT.KBP310G" H 3880 1640 50  0001 C CNN
 F 3 "" H 3880 1640 50  0001 C CNN
 	1    4245 1175
-	1    0    0    -1
+	1    0    0    1
 $EndComp
 Wire Wire Line
@@
 Wire Wire Line
 	5370 1000 5370 1050
-$Comp
-L MenRed_Library_DIODE:D.SMT.1N4007.SOD-123 D3
-U 1 1 613C6FDD
-P 6630 1420
-F 0 "D3" H 6840 1545 50  0000 C CNN
-F 1 "1N4007" H 6870 1470 50  0000 C CNN
-F 2 "MenRed_Library_DIODE:D.SMT.1N4007.SOD-123" H 6580 1270 50  0001 C CNN
-F 3 "" H 6630 1420 50  0001 C CNN
-	1    6630 1420
-	1    0    0    -1
-$EndComp
 $Comp
 L MenRed_Library_RES:RES.SMT.10K.1206 R26
@@
 U 1 1 6187B2C5
 P 7330 1400
-F 0 "TR1" H 7330 2047 50  0000 C CNN
-F 1 "EE16L.JY161150-8W" H 7330 1956 50  0000 C CNN
+F 0 "TR1" H 7075 1685 50  0000 C CNN
+F 1 "EE16L.JY161150-8W" H 7395 1175 50  0000 C CNN
 F 2 "MenRed_Library_L:L.DIP.TRANS.EE16L-5W" H 7330 1400 60  0001 C CNN
 F 3 "" H 7330 1400 60  0000 C CNN
@@
 $EndComp
 Wire Wire Line
-	5965 1000 7130 1000
+	5965 1000 6820 1000
 Wire Wire Line
 	6780 1420 7030 1420
@@
 	8145 1000 8220 1000
 Wire Wire Line
-	7530 1400 8145 1400
+	7530 1400 7620 1400
 Wire Wire Line
 	8635 1400 8635 1360
@@
 P 5330 2615
 F 0 "R8" V 5415 1925 50  0000 L CNN
-F 1 "10R.0805" V 5420 2055 50  0000 L CNN
+F 1 "NC" V 5420 2055 50  0000 L CNN
 F 2 "MenRed_Library_RES:RES.SMT.0805" H 5243 2526 60  0001 C CNN
 F 3 "" H 5330 2615 60  0000 C CNN
@@
 P 5220 2620
 F 0 "R7" V 5215 2045 50  0000 L CNN
-F 1 "10R.0805" V 5215 2180 50  0000 L CNN
+F 1 "3.6K.0805" V 5215 2180 50  0000 L CNN
 F 2 "MenRed_Library_RES:RES.SMT.0805" H 5133 2531 60  0001 C CNN
 F 3 "" H 5220 2620 60  0000 C CNN
@@
 P 5495 2620
 F 0 "R10" V 5470 3230 50  0000 L CNN
-F 1 "10R.0805" V 5470 2815 50  0000 L CNN
+F 1 "1R6.0805" V 5470 2815 50  0000 L CNN
 F 2 "MenRed_Library_RES:RES.SMT.0805" H 5408 2531 60  0001 C CNN
 F 3 "" H 5495 2620 60  0000 C CNN
@@
 P 5595 2625
 F 0 "R11" V 5645 3135 50  0000 L CNN
-F 1 "10R.0805" V 5650 2720 50  0000 L CNN
+F 1 "1R6.0805" V 5650 2720 50  0000 L CNN
 F 2 "MenRed_Library_RES:RES.SMT.0805" H 5508 2536 60  0001 C CNN
 F 3 "" H 5595 2625 60  0000 C CNN
@@
 	11560 6505 11600 6505
 Wire Wire Line
-	3845 1225 3845 885
-Wire Wire Line
-	3845 885  3650 885
-Wire Wire Line
 	3650 885  3645 885
-Wire Wire Line
-	3845 1225 3995 1225
-Wire Wire Line
-	3875 1125 3875 1525
-Wire Wire Line
-	3875 1125 3995 1125
-Wire Wire Line
-	3875 1525 3650 1525
 $Comp
 L MenRed_Library_RES:RES.SMT.10K.0603 R31
@@
 Text Label 12325 6605 0    50   ~ 0
 SW3
+Wire Wire Line
+	3995 1125 3905 1125
+Wire Wire Line
+	3905 1125 3905 885
+Wire Wire Line
+	3650 885  3905 885
+Wire Wire Line
+	3995 1225 3905 1225
+Wire Wire Line
+	3905 1225 3905 1525
+Wire Wire Line
+	3650 1525 3905 1525
+$Comp
+L MenRed_Library_DIODE:D.SMT.1N4007.SOD-123 D3
+U 1 1 613C6FDD
+P 6630 1420
+F 0 "D3" H 6840 1545 50  0000 C CNN
+F 1 "1N4007" H 6870 1470 50  0000 C CNN
+F 2 "MenRed_Library_DIODE:D.SMT.1N4007.SOD-123" H 6580 1270 50  0001 C CNN
+F 3 "" H 6630 1420 50  0001 C CNN
+	1    6630 1420
+	1    0    0    -1
+$EndComp
+$Comp
+L MenRed_Library_CAP:CAP.DIP.X.0.1uF.275V CY3
+U 1 1 6035E0A3
+P 7015 835
+F 0 "CY3" V 6810 760 50  0000 L CNN
+F 1 "2.2nF.250V" V 6885 505 50  0000 L CNN
+F 2 "MenRed_Library_CAP:CAP.DIP.Y.102M／250V" H 6865 835 60  0001 C CNN
+F 3 "" H 6865 835 60  0000 C CNN
+	1    7015 835
+	0    1    1    0
+$EndComp
+$Comp
+L MenRed_Library_CAP:CAP.DIP.X.0.1uF.275V CY4
+U 1 1 60362652
+P 7315 835
+F 0 "CY4" V 7110 760 50  0000 L CNN
+F 1 "2.2nF.250V" V 7185 675 50  0000 L CNN
+F 2 "MenRed_Library_CAP:CAP.DIP.Y.102M／250V" H 7165 835 60  0001 C CNN
+F 3 "" H 7165 835 60  0000 C CNN
+	1    7315 835
+	0    1    1    0
+$EndComp
+Wire Wire Line
+	6865 835  6820 835
+Wire Wire Line
+	6820 835  6820 1000
+Connection ~ 6820 1000
+Wire Wire Line
+	6820 1000 7130 1000
+Wire Wire Line
+	7465 835  7620 835
+Wire Wire Line
+	7620 835  7620 1400
+Connection ~ 7620 1400
+Wire Wire Line
+	7620 1400 8145 1400
+$Comp
+L MenRed_Library_DIODE:D.LED.SMT.BL-HG635A-TRB-0805 LED1
+U 1 1 605F1A42
+P 13690 885
+F 0 "LED1" H 13517 889 50  0000 R CNN
+F 1 "BL-HG635A" H 13517 980 50  0000 R CNN
+F 2 "MenRed_Library_DIODE:D.BL-HG635A-TRB-LED" H 13740 535 50  0001 C CNN
+F 3 "" V 13690 890 50  0001 C CNN
+	1    13690 885
+	-1   0    0    1
+$EndComp
+$Comp
+L MenRed_Library_RES:RES.SMT.10K.0603 R34
+U 1 1 605F47C8
+P 13690 1320
+F 0 "R34" H 13555 1280 50  0000 C CNN
+F 1 "39K.0603" H 13665 1420 50  0000 C CNN
+F 2 "MenRed_Library_RES:RES.SMT.0603" H 13690 1320 60  0001 C CNN
+F 3 "" H 13690 1320 60  0000 C CNN
+	1    13690 1320
+	0    -1   -1   0
+$EndComp
+Wire Wire Line
+	13690 1085 13690 1170
+Wire Wire Line
+	13690 785  13690 755
+$Comp
+L power:+3.3V #PWR014
+U 1 1 60690587
+P 13690 755
+F 0 "#PWR014" H 13690 605 50  0001 C CNN
+F 1 "+3.3V" H 13610 905 50  0000 L CNN
+F 2 "" H 13690 755 50  0001 C CNN
+F 3 "" H 13690 755 50  0001 C CNN
+	1    13690 755
+	1    0    0    -1
+$EndComp
+$Comp
+L power:GND #PWR015
+U 1 1 60690E97
+P 13690 1510
+F 0 "#PWR015" H 13690 1260 50  0001 C CNN
+F 1 "GND" H 13695 1337 50  0000 C CNN
+F 2 "" H 13690 1510 50  0001 C CNN
+F 3 "" H 13690 1510 50  0001 C CNN
+	1    13690 1510
+	1    0    0    -1
+$EndComp
+Wire Wire Line
+	13690 1470 13690 1510
 $EndSCHEMATC
